File: Blimp_PCB_Stable/Blimp_PCB_V1.kicad_sch (KiCad schematic)
At the start: 13 parts, among them J1 S8B-PH-K-S, J2 S4B-XH-A

Commit message: Relabel, Fix 3D models, starting to remap not done yet
Parts:
- added R1: 30K, Capacitor_SMD:C_0603_1608Metric_Pad1.08x0.95mm_HandSolder, symbol Device:R
- added R2: 7.5K, Capacitor_SMD:C_0603_1608Metric_Pad1.08x0.95mm_HandSolder, symbol Device:R
- J1: footprint JST Connector:JST_SH_SM08B-SRSS-TB_1x08-1MP_P1.00mm_Horizontal -> Connector_JST:JST_SH_BM08B-SRSS-TB_1x08-1MP_P1.00mm_Vertical
Connections:
- net BV: now also R1.1; no longer P5.1
- net GND: now also R2.2
- new net: P5.1, R1.2, R2.1
Other:
- moved on the sheet: P5

Commit message: Fixed orientations, added in traces, fixed everything its perfect
Parts:
- added P2: ~, TerminalBlock_Phoenix:TerminalBlock_Phoenix_MKDS-1,5-2_1x02_P5.00mm_Horizontal, symbol Shorting Pints:Shorting_Pins
- P1: footprint Pins:PWM -> Connector_JST:JST_XH_B2B-XH-A_1x02_P2.50mm_Vertical
- P3: footprint PINS:Shorting Pins -> Connector_JST:JST_XH_B2B-XH-A_1x02_P2.50mm_Vertical
- P9: footprint PINS:Latching Pins -> TerminalBlock_Phoenix:TerminalBlock_Phoenix_MKDS-1,5-2_1x02_P5.00mm_Horizontal
- U3: footprint Pins:PWM -> Connector_JST:JST_XH_S2B-XH-A_1x02_P2.50mm_Horizontal
Connections:
- net +5V: now also P1.1 (5V), P8.2 (5V); no longer P1.2 (5V)
- net BV: now also B1.3, P9.2, P2.2; no longer B1.4, P9.1
- net GND: now also B1.4, P1.2 (GND), P9.1, U3.2, P2.1; no longer B1.3, P1.3 (GND), P9.2, U3.3
- net at U3.1: now also P8.3 (SDA.5)
- no-connect marks 34 -> 32

Commit message: Merged Arik stable update into main
Parts:
- removed J2: S4B-XH-A, S4B_XH_A:JST_S4B-XH-A, symbol S4B-XH-A:S4B-XH-A
- removed P2: ~, TerminalBlock_Phoenix:TerminalBlock_Phoenix_MKDS-1,5-2_1x02_P5.00mm_Horizontal, symbol Shorting Pints:Shorting_Pins
- removed R1: 30K, Capacitor_SMD:C_0603_1608Metric_Pad1.08x0.95mm_HandSolder, symbol Device:R
- removed R2: 7.5K, Capacitor_SMD:C_0603_1608Metric_Pad1.08x0.95mm_HandSolder, symbol Device:R
- added P2: ~, PINS:PWM, symbol PWM:PWM
- J1: footprint Connector_JST:JST_SH_BM08B-SRSS-TB_1x08-1MP_P1.00mm_Vertical -> JST Connector:S8B-PH-K-S
- P1: footprint Connector_JST:JST_XH_B2B-XH-A_1x02_P2.50mm_Vertical -> PINS:PWM
- P3: footprint Connector_JST:JST_XH_B2B-XH-A_1x02_P2.50mm_Vertical -> PINS:Shorting Pins
- P4: footprint Pins:PWM -> PINS:PWM
- P9: footprint TerminalBlock_Phoenix:TerminalBlock_Phoenix_MKDS-1,5-2_1x02_P5.00mm_Horizontal -> PINS:Latching Pins
- U3: footprint Connector_JST:JST_XH_S2B-XH-A_1x02_P2.50mm_Horizontal -> PINS:PWM
Connections:
- net +5V: now also P1.2 (5V), P2.2 (5V); no longer P1.1 (5V), P8.2 (5V)
- net BV: now also B1.4, P5.1, P9.1; no longer B1.3, P9.2
- net GND: now also B1.3, P1.3 (GND), P9.2, U3.3, P2.3 (GND); no longer B1.4, P1.2 (GND), P9.1, U3.2
- net at U3.1: no longer P8.3 (SDA.5)
- new net: P8.3 (SDA.5), U3.2
- no-connect marks 32 -> 35
Other:
- moved on the sheet: P4, P5

Commit message: Arik stable update
Parts:
- removed P2: ~, PINS:PWM, symbol PWM:PWM
- added J2: S4B-XH-A, S4B_XH_A:JST_S4B-XH-A, symbol S4B-XH-A:S4B-XH-A
- added P2: ~, TerminalBlock_Phoenix:TerminalBlock_Phoenix_MKDS-1,5-2_1x02_P5.00mm_Horizontal, symbol Shorting Pints:Shorting_Pins
- added R1: 30K, Capacitor_SMD:C_0603_1608Metric_Pad1.08x0.95mm_HandSolder, symbol Device:R
- added R2: 7.5K, Capacitor_SMD:C_0603_1608Metric_Pad1.08x0.95mm_HandSolder, symbol Device:R
- J1: footprint JST Connector:S8B-PH-K-S -> Connector_JST:JST_SH_BM08B-SRSS-TB_1x08-1MP_P1.00mm_Vertical
- P1: footprint PINS:PWM -> Connector_JST:JST_XH_B2B-XH-A_1x02_P2.50mm_Vertical
- P3: footprint PINS:Shorting Pins -> Connector_JST:JST_XH_B2B-XH-A_1x02_P2.50mm_Vertical
- P4: footprint PINS:PWM -> Pins:PWM
- P9: footprint PINS:Latching Pins -> TerminalBlock_Phoenix:TerminalBlock_Phoenix_MKDS-1,5-2_1x02_P5.00mm_Horizontal
- U3: footprint PINS:PWM -> Connector_JST:JST_XH_S2B-XH-A_1x02_P2.50mm_Horizontal
Connections:
- net +5V: now also P1.1 (5V), P8.2 (5V), J2.1; no longer P1.2 (5V)
- net BV: now also B1.3, P9.2, P2.2, R1.1; no longer B1.4, P5.1, P9.1
- net GND: now also B1.4, P1.2 (GND), P8.25 (GND), P8.9 (GND), P9.1, U3.2, J2.2, P2.1, R2.2; no longer B1.3, P1.3 (GND), P8.6 (GND), P9.2, U3.3
- net at U3.1: now also P8.3 (SDA.5)
- net at P8.10 (TXD.0): now also J2.4
- net at P8.8 (RXD.0): now also J2.3
- new net: P5.1, R1.2, R2.1
- no-connect marks 35 -> 31
Other:
- moved on the sheet: P4, P5

Commit message: Fixed all the problems
Parts:
- J2: footprint S4B_XH_A:JST_S4B-XH-A -> S4B-XH-A:JST_S4B-XH-A
Other:
- moved on the sheet: J2
Changed lines of the file:
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@@
 	)
 	(junction
-		(at 152.4 110.49)
+		(at 152.4 111.76)
 		(diameter 0)
 		(color 0 0 0 0)
@@
 	(wire
 		(pts
-			(xy 173.99 137.16) (xy 173.99 115.57)
+			(xy 173.99 137.16) (xy 173.99 116.84)
 		)
 		(stroke
@@
 	(wire
 		(pts
-			(xy 152.4 110.49) (xy 177.8 110.49)
+			(xy 152.4 111.76) (xy 177.8 111.76)
 		)
 		(stroke
@@
 	(wire
 		(pts
-			(xy 160.02 113.03) (xy 177.8 113.03)
+			(xy 160.02 114.3) (xy 177.8 114.3)
 		)
 		(stroke
@@
 	(wire
 		(pts
-			(xy 173.99 115.57) (xy 177.8 115.57)
+			(xy 173.99 116.84) (xy 177.8 116.84)
 		)
 		(stroke
@@
 	(wire
 		(pts
-			(xy 177.8 118.11) (xy 177.8 142.24)
+			(xy 177.8 119.38) (xy 177.8 142.24)
 		)
 		(stroke
@@
 	(wire
 		(pts
-			(xy 160.02 120.65) (xy 160.02 113.03)
+			(xy 160.02 120.65) (xy 160.02 114.3)
 		)
 		(stroke
@@
 	(symbol
 		(lib_id "S4B-XH-A:S4B-XH-A")
-		(at 187.96 115.57 0)
+		(at 187.96 116.84 0)
 		(unit 1)
 		(exclude_from_sim no)
@@
 		(dnp no)
 		(property "Reference" "J2"
-			(at 187.96 112.776 0)
+			(at 187.96 114.046 0)
 			(effects
 				(font
@@
 		)
 		(property "Value" "S4B-XH-A"
-			(at 187.452 116.332 0)
+			(at 187.452 117.602 0)
 			(effects
 				(font
@@
 			)
 		)
-		(property "Footprint" "S4B_XH_A:JST_S4B-XH-A"
-			(at 187.96 115.57 0)
+		(property "Footprint" "S4B-XH-A:JST_S4B-XH-A"
+			(at 187.96 116.84 0)
 			(effects
 				(font
@@
 		)
 		(property "Datasheet" ""
-			(at 187.96 115.57 0)
+			(at 187.96 116.84 0)
 			(effects
 				(font
@@
 		)
 		(property "Description" "To Lidar"
-			(at 191.262 119.38 0)
+			(at 191.262 120.65 0)
 			(effects
 				(font
@@
 		)
 		(property "MANUFACTURER" "JST"
-			(at 187.96 115.57 0)
+			(at 187.96 116.84 0)
 			(effects
 				(font
@@
 	)
 	(symbol
-		(lib_name "Berry_IMU_1")
 		(lib_id "Berry_IMU:Berry_IMU")
 		(at 92.71 74.93 0)

Commit message: fixed DRC and footprint library erros
Parts:
- B1: footprint JST Connector:XT30 -> XT30:XT30
- J2: footprint S4B-XH-A:JST_S4B-XH-A -> S4B_XH_A:JST_S4B-XH-A
- P8: footprint Blimp Library:Orange_Pi_5B -> Orange_Pi_5B:Orange_Pi_5B
- U3: footprint Connector_JST:JST_XH_S2B-XH-A_1x02_P2.50mm_Horizontal -> JST Connector:JST_XH_S2B-XH-A_1x02_P2.50mm_Horizontal
Changed lines of the file:
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@@
 			)
 		)
-		(property "Footprint" "Connector_JST:JST_XH_S2B-XH-A_1x02_P2.50mm_Horizontal"
+		(property "Footprint" "JST Connector:JST_XH_S2B-XH-A_1x02_P2.50mm_Horizontal"
 			(at 146.05 68.58 0)
 			(effects
@@
 			)
 		)
-		(property "Footprint" "S4B-XH-A:JST_S4B-XH-A"
+		(property "Footprint" "S4B_XH_A:JST_S4B-XH-A"
 			(at 187.96 116.84 0)
 			(effects
@@
 			)
 		)
-		(property "Footprint" "JST Connector:XT30"
+		(property "Footprint" "XT30:XT30"
 			(at 203.2 100.33 0)
 			(effects
@@
 			)
 		)
-		(property "Footprint" "Blimp Library:Orange_Pi_5B"
+		(property "Footprint" "Orange_Pi_5B:Orange_Pi_5B"
 			(at 91.948 100.838 0)
 			(effects
